File: Hardware/DigitalLevel.kicad_pcb (KiCad board)
At the start: 2 copper layers, 70 x 70 mm, 34 parts, among them J1 Conn_ARM_SWD_TagConnect_TC2030, J2 AYF531035, SW1 SKRKAHE020, SW2 SKRKAHE020, U1 MAX16150A, U2 TPS60243DGKT, U3 STM32L031K6Ux, U4 LIS2DTW12TR

Commit message: Swap MCU to STM32C0
Parts:
- removed C7, C8: 100nF, Capacitor_SMD:C_0402_1005Metric
- added TP1: TestPoint, TestPoint:TestPoint_Pad_D1.0mm, F.Cu at (120.0, 77.2)
- added TP10: TestPoint, TestPoint:TestPoint_Pad_D1.0mm, F.Cu at (140.0, 124.0)
- added TP11: TestPoint, TestPoint:TestPoint_Pad_D1.0mm, F.Cu at (136.0, 120.0)
- added TP2: TestPoint, TestPoint:TestPoint_Pad_D1.0mm, F.Cu at (119.0, 89.6)
- added TP3: TestPoint, TestPoint:TestPoint_Pad_D1.0mm, F.Cu at (125.8, 82.2)
- added TP4: TestPoint, TestPoint:TestPoint_Pad_D1.0mm, F.Cu at (124.2, 81.4)
- added TP5: TestPoint, TestPoint:TestPoint_Pad_D1.0mm, F.Cu at (135.6, 112.2)
- added TP6: TestPoint, TestPoint:TestPoint_Pad_D1.0mm, F.Cu at (134.0, 110.6)
- added TP7: TestPoint, TestPoint:TestPoint_Pad_D1.0mm, F.Cu at (133.0, 108.2)
- added TP8: TestPoint, TestPoint:TestPoint_Pad_D1.0mm, F.Cu at (138.0, 122.0)
- added TP9: TestPoint, TestPoint:TestPoint_Pad_D1.0mm, F.Cu at (142.0, 126.0)
- U3: value STM32L031K6Ux -> STM32C011F4Ux; footprint Package_DFN_QFN:QFN-32-1EP_5x5mm_P0.5mm_EP3.45x3.45mm -> Package_DFN_QFN:ST_UFQFPN-20_3x3mm_P0.5mm
- moved R7 14.7 mm to (130.2, 114.0), turned to 90 degrees
- moved R5 12.4 mm to (130.2, 118.4), turned to -90 degrees
- moved C5 5.51 mm to (125.0, 108.8), turned to 180 degrees
- moved C9 5.15 mm to (122.5, 110.0), turned to 180 degrees
- moved R8 2.41 mm to (132.0, 118.4)
- moved C6 2.34 mm to (125.0, 109.8), turned to 180 degrees
- moved R6 2.11 mm to (132.0, 114.0), turned to 90 degrees
- moved C15 1.25 mm to (145.5, 127.8)
Connections:
- U3 pad 1: +3V0 -> /ACC_INT
- U3 pad 10: /nPWR_INT -> unconnected-(U3-PA5-Pad10)
- U3 pad 11: unconnected-(U3-PA5-Pad11) -> /FUNC_BUTTON
- U3 pad 13: unconnected-(U3-PA7-Pad13) -> /DISP_EN
- U3 pad 14: unconnected-(U3-PB0-Pad14) -> /DISP_CS
- U3 pad 15: unconnected-(U3-PB1-Pad15) -> /DISP_MOSI
- U3 pad 16: unconnected-(U3-PB2-Pad16) -> /SWDIO
- U3 pad 17: +3V0 -> /SWCLK
- U3 pad 18: unconnected-(U3-PA8-Pad18) -> /DISP_SCLK
- U3 pad 19: unconnected-(U3-PA9-Pad19) -> /SCL
- U3 pad 2: unconnected-(U3-PC14-Pad2) -> +3V0
- U3 pad 20: unconnected-(U3-PA10-Pad20) -> /SDA
- U3 pad 3: unconnected-(U3-PC15-Pad3) -> GND
- U3 pad 5: +3V0 -> unconnected-(U3-PA0-Pad5)
- U3 pad 6: unconnected-(U3-PA0-Pad6) -> /nPWR_INT
- U3 pad 7: unconnected-(U3-PA1-Pad7) -> /nPWR_OFF
- U3 pad 9: /nPWR_OFF -> unconnected-(U3-PA4-Pad9)
Routing:
- net +3V0: track 176.5 -> 158.9 mm
- net /DISP_SCLK: track 33.3 -> 42.4 mm, vias 0 -> 2
- net /DISP_EN: track 30.9 -> 36.6 mm, vias 0 -> 2
- net /FUNC_BUTTON: track 56.4 -> 61.9 mm
- net /DISP_CS: track 34.4 -> 38.5 mm
- net GND: track 11.7 -> 15.8 mm, vias 38 -> 44
- net /SWCLK: track 14.5 -> 18.3 mm, vias 0 -> 2
- net /ACC_INT: track 54.9 -> 51.6 mm, vias 4 -> 2
- net /SWDIO: track 18.1 -> 20.6 mm, vias 0 -> 2
- net /nRESET: track 30.8 -> 28.3 mm, vias 3 -> 2
- net /nPWR_OFF: track 40.5 -> 42.2 mm
- net /nPWR_INT: track 41.7 -> 40.2 mm
- net /SCL: track 47.3 -> 48.7 mm
- net /DISP_MOSI: track 38.2 -> 39.6 mm, vias 0 -> 2
- net /SDA: track 47.4 -> 48.5 mm, vias 0 -> 2
Other:
- board text added: "Digital Level Thomas Gonnot 2025-05-16 - v2.0"
- board text removed: "Digital Level Thomas Gonnot 2024-11-13 - v1.0"
