File: Hardware/DigitalLevel.kicad_sch (KiCad schematic)
At the start: 34 parts, among them J1 Conn_ARM_SWD_TagConnect_TC2030, J2 AYF531035, SW1 SKRKAHE020, SW2 SKRKAHE020, U1 MAX16150A, U2 TPS60243DGKT, U3 STM32L031K6Ux, U4 LIS2DTW12TR

Commit message: Swap MCU to STM32C0
Parts:
- removed C7, C8: 100nF, Capacitor_SMD:C_0402_1005Metric, symbol Device:C
- added TP1, TP10, TP11, TP2, TP3, TP4, TP5, TP6, TP7, TP8, TP9: TestPoint, TestPoint:TestPoint_Pad_D1.0mm, symbol Connector:TestPoint
- U3: value STM32L031K6Ux -> STM32C011F4Ux; footprint Package_DFN_QFN:QFN-32-1EP_5x5mm_P0.5mm_EP3.45x3.45mm -> Package_DFN_QFN:ST_UFQFPN-20_3x3mm_P0.5mm; symbol MCU_ST_STM32L0:STM32L031K4Ux -> MCU_ST_STM32C0:STM32C011F4Ux
Connections:
- net +3V0: now also U3.2 (VDD), TP2.1; no longer U3.1 (VDD), U3.17 (VDD), U3.5 (VDDA)
- net ACC_INT: now also U3.1 (PC15), TP7.1; no longer U3.21 (PA11)
- net DISP_CS: now also U3.14 (PA9/PA11), TP8.1; no longer U3.27 (PB4)
- net DISP_EN: now also U3.13 (PA8), TP11.1; no longer U3.25 (PA15)
- net DISP_MOSI: now also U3.15 (PA10/PA12), TP10.1; no longer U3.28 (PB5)
- net DISP_SCLK: now also U3.18 (PB6), TP9.1; no longer U3.26 (PB3)
- net FUNC_BUTTON: now also U3.11 (PA6); no longer U3.29 (PB6)
- net GND: now also U3.3 (VSS); no longer U3.33 (VSS)
- net SCL: now also U3.19 (PB7), TP6.1; no longer U3.32 (PB8)
- net SDA: now also U3.20 (PC14), TP5.1; no longer U3.30 (PB7)
- net SWCLK: now also U3.17 (PA14); no longer U3.24 (PA14)
- net SWDIO: now also U3.16 (PA13); no longer U3.23 (PA13)
- net VPWR: now also TP1.1
- net nPWR_INT: now also U3.6 (PA1), TP3.1; no longer U3.10 (PA4)
- net nPWR_OFF: now also U3.7 (PA2), TP4.1; no longer U3.9 (PA3)
- no-connect marks 20 -> 9
Other:
- note added: "Max. 25mA"
- moved on the sheet: C5, C6, C9, J1
